Commit message: updated urdf and sdf files for comparision

File: ssl_robot_description/urdf/robot.urdf (robot description, URDF)
Before this commit: robot ssl_robot, 86 links, 85 joints
Links:
- link base_plate: geometry collision cylinder length=0.001 radius=0.07
- link sub_wheel_fl_1: mass 0.001 -> 0.0010
- link sub_wheel_fl_10: mass 0.001 -> 0.0010
- link sub_wheel_fl_11: mass 0.001 -> 0.0010
- link sub_wheel_fl_12: mass 0.001 -> 0.0010
- link sub_wheel_fl_13: mass 0.001 -> 0.0010
- link sub_wheel_fl_14: mass 0.001 -> 0.0010
- link sub_wheel_fl_15: mass 0.001 -> 0.0010
- link sub_wheel_fl_16: mass 0.001 -> 0.0010
- link sub_wheel_fl_17: mass 0.001 -> 0.0010
- link sub_wheel_fl_18: mass 0.001 -> 0.0010
- link sub_wheel_fl_19: mass 0.001 -> 0.0010
- link sub_wheel_fl_2: mass 0.001 -> 0.0010
- link sub_wheel_fl_20: mass 0.001 -> 0.0010
- link sub_wheel_fl_3: mass 0.001 -> 0.0010
- link sub_wheel_fl_4: mass 0.001 -> 0.0010
- link sub_wheel_fl_5: mass 0.001 -> 0.0010
- link sub_wheel_fl_6: mass 0.001 -> 0.0010
- link sub_wheel_fl_7: mass 0.001 -> 0.0010
- link sub_wheel_fl_8: mass 0.001 -> 0.0010
- link sub_wheel_fl_9: mass 0.001 -> 0.0010
- link sub_wheel_fr_1: mass 0.001 -> 0.0010
- link sub_wheel_fr_10: mass 0.001 -> 0.0010
- link sub_wheel_fr_11: mass 0.001 -> 0.0010
- link sub_wheel_fr_12: mass 0.001 -> 0.0010
- link sub_wheel_fr_13: mass 0.001 -> 0.0010
- link sub_wheel_fr_14: mass 0.001 -> 0.0010
- link sub_wheel_fr_15: mass 0.001 -> 0.0010
- link sub_wheel_fr_16: mass 0.001 -> 0.0010
- link sub_wheel_fr_17: mass 0.001 -> 0.0010
- link sub_wheel_fr_18: mass 0.001 -> 0.0010
- link sub_wheel_fr_19: mass 0.001 -> 0.0010
- link sub_wheel_fr_2: mass 0.001 -> 0.0010
- link sub_wheel_fr_20: mass 0.001 -> 0.0010
- link sub_wheel_fr_3: mass 0.001 -> 0.0010
- link sub_wheel_fr_4: mass 0.001 -> 0.0010
- link sub_wheel_fr_5: mass 0.001 -> 0.0010
- link sub_wheel_fr_6: mass 0.001 -> 0.0010
- link sub_wheel_fr_7: mass 0.001 -> 0.0010
- link sub_wheel_fr_8: mass 0.001 -> 0.0010
- link sub_wheel_fr_9: mass 0.001 -> 0.0010
- link sub_wheel_rl_1: mass 0.001 -> 0.0010
- link sub_wheel_rl_10: mass 0.001 -> 0.0010
- link sub_wheel_rl_11: mass 0.001 -> 0.0010
- link sub_wheel_rl_12: mass 0.001 -> 0.0010
- link sub_wheel_rl_13: mass 0.001 -> 0.0010
- link sub_wheel_rl_14: mass 0.001 -> 0.0010
- link sub_wheel_rl_15: mass 0.001 -> 0.0010
- link sub_wheel_rl_16: mass 0.001 -> 0.0010
- link sub_wheel_rl_17: mass 0.001 -> 0.0010
- link sub_wheel_rl_18: mass 0.001 -> 0.0010
- link sub_wheel_rl_19: mass 0.001 -> 0.0010
- link sub_wheel_rl_2: mass 0.001 -> 0.0010
- link sub_wheel_rl_20: mass 0.001 -> 0.0010
- link sub_wheel_rl_3: mass 0.001 -> 0.0010
- link sub_wheel_rl_4: mass 0.001 -> 0.0010
- link sub_wheel_rl_5: mass 0.001 -> 0.0010
- link sub_wheel_rl_6: mass 0.001 -> 0.0010
- link sub_wheel_rl_7: mass 0.001 -> 0.0010
- link sub_wheel_rl_8: mass 0.001 -> 0.0010
- link sub_wheel_rl_9: mass 0.001 -> 0.0010
- link sub_wheel_rr_1: mass 0.001 -> 0.0010
- link sub_wheel_rr_10: mass 0.001 -> 0.0010
- link sub_wheel_rr_11: mass 0.001 -> 0.0010
- link sub_wheel_rr_12: mass 0.001 -> 0.0010
- link sub_wheel_rr_13: mass 0.001 -> 0.0010
- link sub_wheel_rr_14: mass 0.001 -> 0.0010
- link sub_wheel_rr_15: mass 0.001 -> 0.0010
- link sub_wheel_rr_16: mass 0.001 -> 0.0010
- link sub_wheel_rr_17: mass 0.001 -> 0.0010
- link sub_wheel_rr_18: mass 0.001 -> 0.0010
- link sub_wheel_rr_19: mass 0.001 -> 0.0010
- link sub_wheel_rr_2: mass 0.001 -> 0.0010
- link sub_wheel_rr_20: mass 0.001 -> 0.0010
- link sub_wheel_rr_3: mass 0.001 -> 0.0010
- link sub_wheel_rr_4: mass 0.001 -> 0.0010
- link sub_wheel_rr_5: mass 0.001 -> 0.0010
- link sub_wheel_rr_6: mass 0.001 -> 0.0010
- link sub_wheel_rr_7: mass 0.001 -> 0.0010
- link sub_wheel_rr_8: mass 0.001 -> 0.0010
- link sub_wheel_rr_9: mass 0.001 -> 0.0010
- link wheel_fl: mass 0.05 -> 0.0050
- link wheel_fr: mass 0.05 -> 0.0050
- link wheel_rl: mass 0.05 -> 0.0050
- link wheel_rr: mass 0.05 -> 0.0050
Joints:
- joint base_joint: origin xyz=0 0 0.1 rpy=0 0 0 -> xyz=0 0 0.05 rpy=0 0 0
