Commit message: better robot simulation and control

File: ssl_robot_description/urdf/ssl_robot.xacro (robot description, xacro)
@@ -1,42 +1,32 @@
 <?xml version="1.0"?>
 <robot name="ssl_robot" xmlns:xacro="http://www.ros.org/wiki/xacro">
-  <!-- Constants for robot dimensions -->
-  <xacro:property name="PI" value="3.1415926535897931" />
-  <xacro:property name="over_ground" value="0.02" />
-  <xacro:property name="platform_height" value="0.015" />
-  <xacro:property name="ground_clearance" value="0.005" />
-  <xacro:property name="base_height" value="0.005" />
-  <xacro:property name="base_radius" value="0.07" />
-  <xacro:property name="robot_height" value="0.15" />
-  <xacro:property name="friction" value="0.2" />
-  <!-- Import all Gazebo-customization elements, including Gazebo colors -->
+  <xacro:property name="ground_clearance" value="0.002" />
+  <xacro:property name="base_height" value="0.145" />
+  <xacro:property name="base_radius" value="0.09" />
   <xacro:include filename="$(find ssl_robot_description)/urdf/ssl_robot.gazebo" />
-  <!-- Import Rviz colors -->
   <xacro:include filename="$(find ssl_robot_description)/urdf/materials.xacro" />
-  <!-- Import wheel macros -->
-  <xacro:include filename="$(find ssl_robot_description)/urdf/wheel.xacro" />
-  <!-- Base Link -->
+  <xacro:include filename="$(find ssl_robot_description)/urdf/wheel2.xacro" />
   <link name="base_link">
   </link>
   <link name="base_plate">
    <inertial>
-     <origin xyz="0 0 ${robot_height/2}" rpy="0 0 0"/>
-     <mass value="2.5"/>
+     <origin xyz="0 0 ${base_height/2+ground_clearance-0.02}" rpy="0 0 0"/>
+     <mass value="2.50" />
 <!--
-     <inertia ixx="30.9250"  ixy="-0.2628"  ixz="-0.0222" iyy="33.5471" iyz="0.8517" izz="33.0306" />
+     <inertia ixx="0.0008896" ixy="0" ixz="0" iyy="0.0008896" iyz="0" izz="0.0009031" />
 -->
-     <inertia ixx="0.0097" ixy="0"  ixz="0" iyy="0.0097" iyz="0" izz="0.0101" />
+     <inertia ixx="0.0008896" ixy="0" ixz="0" iyy="0.0008896" iyz="0" izz="0.0009031" />
    </inertial>
    <visual>
-     <origin xyz="0 0 ${over_ground+base_height/2+ground_clearance}" rpy="0 0 0" />
+     <origin xyz="0 0 0" rpy="0 0 -1.5707"/>
      <geometry>
+       <mesh filename="package://ssl_robot_description/meshes/HBG-Roboter-now.stl"/>
+<!--
        <cylinder radius="${base_radius}" length="${base_height}"/>
+-->
      </geometry>
-     <material name="Cyan">
-       <color rgba="0 1.0 1.0 1.0"/>
-     </material>
    </visual>
    <collision>
-     <origin xyz="0 0 ${over_ground+base_height/2+ground_clearance}" rpy="0 0 0" />
+     <origin xyz="0 0 ${base_height/2+ground_clearance}" rpy="0 0 0"/>
      <geometry>
        <cylinder radius="${base_radius}" length="${base_height}"/>
@@ -48,26 +38,6 @@
     <child link="base_plate" />
     <axis xyz="1 0 0" />
+    <origin xyz="0 0 0.1" rpy="0 0 0" />
   </joint>
-<!--
-  <link name="platform">
-   <visual>
-     <origin xyz="0 0 ${platform_height/2}" rpy="0 0 0" />
-     <geometry>
-       <cylinder radius="0.05" length="${platform_height}"/>
-     </geometry>
-   </visual>
-   <collision>
-     <origin xyz="0 0 ${platform_height/2}" rpy="0 0 0" />
-     <geometry>
-       <cylinder radius="0.05" length="${platform_height}"/>
-     </geometry>
-   </collision>
-  </link>
-  <joint name="platform_joint" type="fixed">
-    <parent link="base_link" />
-    <child link="platform" />
-    <axis xyz="1 0 0" />
-  </joint>
--->
   <xacro:wheel suffix="fr" parent="base_plate" origin_x="0.5" origin_y="-0.8660" rotation="-1.0472" />
   <xacro:wheel suffix="fl" parent="base_plate" origin_x="0.5" origin_y="0.8660" rotation="1.0472" />

File: ssl_robot_description/urdf/wheel.xacro (robot description, xacro)
@@ -1,55 +1,22 @@
 <?xml version="1.0"?>
 <robot xmlns:xacro="http://www.ros.org/wiki/xacro">
-  <xacro:property name="wheel_radius" value="0.025" />
-  <xacro:property name="motor_height" value="0.04" />
-  <xacro:property name="motor_thickness" value="0.02" />
-  <xacro:property name="wheel_thickness" value="0.01" />
-  <xacro:property name="robot_wheel_radius" value="0.08" />
+  <xacro:property name="wheel_radius" value="0.027" />
+  <xacro:property name="wheel_thickness" value="0.015" />
+  <xacro:property name="robot_wheel_radius" value="0.075" />
   <xacro:macro name="wheel" params="suffix parent origin_x origin_y rotation">
-    <link name="motor_${suffix}">
+    <link name="wheel_${suffix}">
       <inertial>
-        <origin xyz="0 0 0" rpy="0 0 0" />
-        <mass value="1" />
-<!--
-        <inertia ixx="5.7332" ixy="0" ixz="0" iyy="5.7332" iyz="0" izz="10.4076" />
--->
-<!--
-        <inertia ixx="0.000016667" ixy="0" ixz="0" iyy="0.000016667" iyz="0" izz="0.000026667" />
--->
-        <inertia ixx="1" ixy="0" ixz="0" iyy="1" iyz="0" izz="1" />
+        <origin xyz="0.005 0 0" rpy="0 1.5707 0" />
+        <mass value="0.10" />
+        <inertia ixx="0.000016" ixy="0" ixz="0" iyy="0.000016" iyz="0" izz="0.000031" />
       </inertial>
-      <visual>
-        <origin xyz="0 0 0" rpy="0 0 0" />
+      <visual name="wheel-visual" >
+        <origin xyz="0 0 0" rpy="0 1.5707 0" />
         <geometry>
-          <box size="${motor_thickness} ${motor_height} ${motor_height}" />
+          <mesh filename="package://ssl_robot_description/meshes/UBG-Rad.stl"/>
         </geometry>
       </visual>
-      <collision>
-        <origin xyz="0 0 0" rpy="0 0 0" />
-        <geometry>
-          <box size="${motor_thickness} ${motor_height} ${motor_height}" />
-        </geometry>
-      </collision>
-    </link>
-    <link name="wheel_${suffix}">
-      <inertial>
-        <origin xyz="0 0 0.00" rpy="0 0 0" />
-        <mass value="1" />
-<!--
-        <inertia ixx="5.7332" ixy="0" ixz="0" iyy="5.7332" iyz="0" izz="10.4076" />
--->
-<!--
-        <inertia ixx="0.000016458" ixy="0" ixz="0" iyy="0.000016458" iyz="0" izz="0.000031250" />
--->
-        <inertia ixx="1" ixy="0" ixz="0" iyy="1" iyz="0" izz="1" />
-      </inertial>
-      <visual>
-        <origin xyz="0 0 0" rpy="0 1.5707 0" />
-        <geometry>
-          <cylinder radius="${wheel_radius}" length="${wheel_thickness}" />
-        </geometry>
-      </visual>
-      <collision>
-        <origin xyz="0 0 0" rpy="0 1.5707 0" />
+      <collision name="wheel">
+        <origin xyz="0.005 0 0" rpy="0 1.5707 0" />
         <geometry>
           <cylinder radius="${wheel_radius}" length="${wheel_thickness}" />
@@ -57,21 +24,30 @@
       </collision>
     </link>
+    <link name="motor_${suffix}">
+      <inertial>
+        <origin xyz="${robot_wheel_radius-wheel_thickness-0.005} 0 ${wheel_radius}" rpy="0 0 0" />
+        <mass value="0.10" />
+        <inertia ixx="0.000042" ixy="0" ixz="0" iyy="0.000022" iyz="0" izz="0.000022" />
+      </inertial>
+      <visual>
+        <origin xyz="${robot_wheel_radius-wheel_thickness-0.0005} 0 ${wheel_radius}" rpy="0 0 0" />
+        <geometry>
+          <box size="0.001 ${wheel_radius*2} ${wheel_radius*2}" />
+        </geometry>
+      </visual>
+    </link>
     <joint name="base_wheel_${suffix}" type="continuous">
       <parent link="motor_${suffix}" />
       <child link="wheel_${suffix}" />
       <axis xyz="1 0 0" />
-      <origin xyz="${wheel_thickness/2+motor_thickness/2+0.001} 0 ${-ground_clearance-base_height}" rpy="0 0 0" />
-<!--
-      <dynamics damping="0.7" />
--->
+      <origin xyz="${robot_wheel_radius} 0 ${wheel_radius-ground_clearance}" rpy="0 0 0" />
     </joint>
-    <joint name="base_motor_${suffix}" type="fixed">
+    <joint name="base_motor_${suffix}" type="revolute">
       <parent link="${parent}" />
       <child link="motor_${suffix}" />
-      <axis xyz="1 0 0" />
-      <origin xyz="${origin_x * (robot_wheel_radius-motor_thickness/2-wheel_thickness/2)}
-                   ${origin_y * (robot_wheel_radius-motor_thickness/2-wheel_thickness/2)}
-                   ${ground_clearance + over_ground + base_height + motor_height/2}"
-              rpy="0 0 ${rotation}" />
+      <axis xyz="0 0 1" />
+      <limit effort="30" velocity="1.0" lower="${rotation}" upper="${rotation}" />
+      <origin xyz="0 0 0"
+              rpy="0 0 0" />
     </joint>
     <transmission name="tran_${suffix}">
@@ -80,5 +56,5 @@
         <hardwareInterface>EffortJointInterface</hardwareInterface>
       </joint>
-      <actuator name="motor_${suffix}">
+      <actuator name="wheel_${suffix}">
         <hardwareInterface>EffortJointInterface</hardwareInterface>
         <mechanicalReduction>1</mechanicalReduction>

Commit message: gazebo SSL robot working now, shared radio server added

File: ssl_robot_description/urdf/ssl_robot.xacro (robot description, xacro)
@@ -2,19 +2,20 @@
 <robot name="ssl_robot" xmlns:xacro="http://www.ros.org/wiki/xacro">
   <xacro:property name="ground_clearance" value="0.002" />
-  <xacro:property name="base_height" value="0.145" />
+  <xacro:property name="base_height" value="0.15" />
   <xacro:property name="base_radius" value="0.09" />
   <xacro:include filename="$(find ssl_robot_description)/urdf/ssl_robot.gazebo" />
   <xacro:include filename="$(find ssl_robot_description)/urdf/materials.xacro" />
-  <xacro:include filename="$(find ssl_robot_description)/urdf/wheel2.xacro" />
+  <xacro:include filename="$(find ssl_robot_description)/urdf/wheel.xacro" />
   <link name="base_link">
   </link>
   <link name="base_plate">
    <inertial>
-     <origin xyz="0 0 ${base_height/2+ground_clearance-0.02}" rpy="0 0 0"/>
-     <mass value="2.50" />
+      <origin xyz="0 0 ${base_height/2+ground_clearance}" rpy="0 0 0"/>
 <!--
-     <inertia ixx="0.0008896" ixy="0" ixz="0" iyy="0.0008896" iyz="0" izz="0.0009031" />
+      <mass value="1.00" />
+      <inertia ixx="0.001233" ixy="0" ixz="0" iyy="0.001233" iyz="0" izz="0.002450" />
 -->
-     <inertia ixx="0.0008896" ixy="0" ixz="0" iyy="0.0008896" iyz="0" izz="0.0009031" />
+      <mass value="5.00" />
+      <inertia ixx="0.015500" ixy="0" ixz="0" iyy="0.015500" iyz="0" izz="0.012250" />
    </inertial>
    <visual>
@@ -22,7 +23,4 @@
      <geometry>
        <mesh filename="package://ssl_robot_description/meshes/HBG-Roboter-now.stl"/>
-<!--
-       <cylinder radius="${base_radius}" length="${base_height}"/>
--->
      </geometry>
    </visual>
@@ -38,5 +36,5 @@
     <child link="base_plate" />
     <axis xyz="1 0 0" />
-    <origin xyz="0 0 0.1" rpy="0 0 0" />
+    <origin xyz="0 0 0.01" rpy="0 0 0" />
   </joint>
   <xacro:wheel suffix="fr" parent="base_plate" origin_x="0.5" origin_y="-0.8660" rotation="-1.0472" />

File: ssl_robot_description/urdf/sub_wheel.xacro (robot description, xacro)
@@ -7,14 +7,12 @@
       <inertial>
         <origin xyz="0 0 0" rpy="0 0 0" />
-        <mass value="0.0010" />
-        <inertia ixx="0.0000000111" ixy="0" ixz="0" iyy="0.0000000111" iyz="0" izz="0.0000000211" />
+<!--
+        <mass value="0.1000" />
+        <inertia ixx="0.0002500521" ixy="0" ixz="0" iyy="0.0002500521" iyz="0" izz="0.0005000000" />
+-->
+        <mass value="0.1000" />
+        <inertia ixx="0.0000625521" ixy="0" ixz="0" iyy="0.0000625521" iyz="0" izz="0.0001250000" />
       </inertial>
-      <visual name="wheel-visual" >
-        <origin xyz="0 0 0" rpy="0 0 0" />
-        <geometry>
-          <cylinder radius="${sub_wheel_radius}" length="${sub_wheel_thickness}" />
-        </geometry>
-      </visual>
-      <collision name="wheel">
+      <collision>
         <origin xyz="0 0 0" rpy="0 0 0" />
         <geometry>
@@ -28,10 +26,5 @@
       <axis xyz="0 0 1" />
       <origin xyz="0.007 ${origin_x} ${origin_y}" rpy="${rotation} 0 0" />
-<!--
-      <dynamics damping="0.0" friction="0.2" />
--->
-<!--
-      <limit effort="30" velocity="1" />
--->
+      <dynamics damping="0.0001" friction="0.0" />
     </joint>
   </xacro:macro>

File: ssl_robot_description/urdf/wheel.xacro (robot description, xacro)
@@ -1,15 +1,20 @@
 <?xml version="1.0"?>
 <robot xmlns:xacro="http://www.ros.org/wiki/xacro">
-  <xacro:property name="wheel_radius" value="0.027" />
+  <xacro:property name="wheel_radius" value="0.025" />
   <xacro:property name="wheel_thickness" value="0.015" />
   <xacro:property name="robot_wheel_radius" value="0.075" />
+  <xacro:include filename="$(find ssl_robot_description)/urdf/sub_wheel.xacro" />
   <xacro:macro name="wheel" params="suffix parent origin_x origin_y rotation">
     <link name="wheel_${suffix}">
       <inertial>
-        <origin xyz="0.005 0 0" rpy="0 1.5707 0" />
-        <mass value="0.10" />
-        <inertia ixx="0.000016" ixy="0" ixz="0" iyy="0.000016" iyz="0" izz="0.000031" />
+        <origin xyz="${wheel_thickness/2} 0 0" rpy="0 1.5707 0" />
+<!--
+        <mass value="0.5000" />
+        <inertia ixx="0.0003218750" ixy="0" ixz="0" iyy="0.0003218750" iyz="0" izz="0.0006250000" />
+-->
+        <mass value="0.5000" />
+        <inertia ixx="0.0012593750" ixy="0" ixz="0" iyy="0.0012593750" iyz="0" izz="0.0025000000" />
       </inertial>
-      <visual name="wheel-visual" >
+      <visual>
         <origin xyz="0 0 0" rpy="0 1.5707 0" />
         <geometry>
@@ -17,38 +22,43 @@
         </geometry>
       </visual>
-      <collision name="wheel">
-        <origin xyz="0.005 0 0" rpy="0 1.5707 0" />
+      <collision>
+        <origin xyz="${wheel_thickness/2} 0 0" rpy="0 1.5707 0" />
         <geometry>
-          <cylinder radius="${wheel_radius}" length="${wheel_thickness}" />
+          <cylinder radius="${wheel_radius}" length="${wheel_thickness}"/>
         </geometry>
       </collision>
     </link>
-    <link name="motor_${suffix}">
-      <inertial>
-        <origin xyz="${robot_wheel_radius-wheel_thickness-0.005} 0 ${wheel_radius}" rpy="0 0 0" />
-        <mass value="0.10" />
-        <inertia ixx="0.000042" ixy="0" ixz="0" iyy="0.000022" iyz="0" izz="0.000022" />
-      </inertial>
-      <visual>
-        <origin xyz="${robot_wheel_radius-wheel_thickness-0.0005} 0 ${wheel_radius}" rpy="0 0 0" />
-        <geometry>
-          <box size="0.001 ${wheel_radius*2} ${wheel_radius*2}" />
-        </geometry>
-      </visual>
-    </link>
     <joint name="base_wheel_${suffix}" type="continuous">
-      <parent link="motor_${suffix}" />
+      <parent link="${parent}" />
       <child link="wheel_${suffix}" />
       <axis xyz="1 0 0" />
-      <origin xyz="${robot_wheel_radius} 0 ${wheel_radius-ground_clearance}" rpy="0 0 0" />
+      <origin xyz="${robot_wheel_radius*origin_x} ${robot_wheel_radius*origin_y} ${wheel_radius-ground_clearance}" rpy="0 0 ${rotation}" />
+      <dynamics damping="0.01" friction="0.0" />
+      <!-- (3m/s / 2*pi*r) * 2 * pi -> 3m/s / r-->
+<!--
+      <limit lower="0" upper="0"
+             effort="1" velocity="${3/wheel_radius}" />
+-->
     </joint>
-    <joint name="base_motor_${suffix}" type="revolute">
-      <parent link="${parent}" />
-      <child link="motor_${suffix}" />
-      <axis xyz="0 0 1" />
-      <limit effort="30" velocity="1.0" lower="${rotation}" upper="${rotation}" />
-      <origin xyz="0 0 0"
-              rpy="0 0 0" />
-    </joint>
+    <xacro:sub_wheel suffix="${suffix}_1" parent="wheel_${suffix}" origin_x="${(wheel_radius-0.005)*1.000000}" origin_y="${(wheel_radius-0.005)*0.000000}" rotation="0.000000" />
+    <xacro:sub_wheel suffix="${suffix}_2" parent="wheel_${suffix}" origin_x="${(wheel_radius-0.005)*0.951057}" origin_y="${(wheel_radius-0.005)*0.309017}" rotation="0.314159" />
+    <xacro:sub_wheel suffix="${suffix}_3" parent="wheel_${suffix}" origin_x="${(wheel_radius-0.005)*0.809017}" origin_y="${(wheel_radius-0.005)*0.587785}" rotation="0.628319" />
+    <xacro:sub_wheel suffix="${suffix}_4" parent="wheel_${suffix}" origin_x="${(wheel_radius-0.005)*0.587785}" origin_y="${(wheel_radius-0.005)*0.809017}" rotation="0.942478" />
+    <xacro:sub_wheel suffix="${suffix}_5" parent="wheel_${suffix}" origin_x="${(wheel_radius-0.005)*0.309017}" origin_y="${(wheel_radius-0.005)*0.951057}" rotation="1.256637" />
+    <xacro:sub_wheel suffix="${suffix}_6" parent="wheel_${suffix}" origin_x="${(wheel_radius-0.005)*0.000000}" origin_y="${(wheel_radius-0.005)*1.000000}" rotation="1.570796" />
+    <xacro:sub_wheel suffix="${suffix}_7" parent="wheel_${suffix}" origin_x="${(wheel_radius-0.005)*-0.309017}" origin_y="${(wheel_radius-0.005)*0.951057}" rotation="1.884956" />
+    <xacro:sub_wheel suffix="${suffix}_8" parent="wheel_${suffix}" origin_x="${(wheel_radius-0.005)*-0.587785}" origin_y="${(wheel_radius-0.005)*0.809017}" rotation="2.199115" />
+    <xacro:sub_wheel suffix="${suffix}_9" parent="wheel_${suffix}" origin_x="${(wheel_radius-0.005)*-0.809017}" origin_y="${(wheel_radius-0.005)*0.587785}" rotation="2.513274" />
+    <xacro:sub_wheel suffix="${suffix}_10" parent="wheel_${suffix}" origin_x="${(wheel_radius-0.005)*-0.951057}" origin_y="${(wheel_radius-0.005)*0.309017}" rotation="2.827433" />
+    <xacro:sub_wheel suffix="${suffix}_11" parent="wheel_${suffix}" origin_x="${(wheel_radius-0.005)*-1.000000}" origin_y="${(wheel_radius-0.005)*0.000000}" rotation="3.141593" />
+    <xacro:sub_wheel suffix="${suffix}_12" parent="wheel_${suffix}" origin_x="${(wheel_radius-0.005)*-0.951057}" origin_y="${(wheel_radius-0.005)*-0.309017}" rotation="3.455752" />
+    <xacro:sub_wheel suffix="${suffix}_13" parent="wheel_${suffix}" origin_x="${(wheel_radius-0.005)*-0.809017}" origin_y="${(wheel_radius-0.005)*-0.587785}" rotation="3.769911" />
+    <xacro:sub_wheel suffix="${suffix}_14" parent="wheel_${suffix}" origin_x="${(wheel_radius-0.005)*-0.587785}" origin_y="${(wheel_radius-0.005)*-0.809017}" rotation="4.084070" />
+    <xacro:sub_wheel suffix="${suffix}_15" parent="wheel_${suffix}" origin_x="${(wheel_radius-0.005)*-0.309017}" origin_y="${(wheel_radius-0.005)*-0.951057}" rotation="4.398230" />
+    <xacro:sub_wheel suffix="${suffix}_16" parent="wheel_${suffix}" origin_x="${(wheel_radius-0.005)*-0.000000}" origin_y="${(wheel_radius-0.005)*-1.000000}" rotation="4.712389" />
+    <xacro:sub_wheel suffix="${suffix}_17" parent="wheel_${suffix}" origin_x="${(wheel_radius-0.005)*0.309017}" origin_y="${(wheel_radius-0.005)*-0.951057}" rotation="5.026548" />
+    <xacro:sub_wheel suffix="${suffix}_18" parent="wheel_${suffix}" origin_x="${(wheel_radius-0.005)*0.587785}" origin_y="${(wheel_radius-0.005)*-0.809017}" rotation="5.340708" />
+    <xacro:sub_wheel suffix="${suffix}_19" parent="wheel_${suffix}" origin_x="${(wheel_radius-0.005)*0.809017}" origin_y="${(wheel_radius-0.005)*-0.587785}" rotation="5.654867" />
+    <xacro:sub_wheel suffix="${suffix}_20" parent="wheel_${suffix}" origin_x="${(wheel_radius-0.005)*0.951057}" origin_y="${(wheel_radius-0.005)*-0.309017}" rotation="5.969026" />
     <transmission name="tran_${suffix}">
       <type>transmission_interface/SimpleTransmission</type>

Commit message: updated gazebo model:
* use inertias from Inventor model, scaled by 10, because 1g mass for
  subwheels instable
* tweaked kp, maxDepth (smoother contact) and friction

File: ssl_robot_description/urdf/ssl_robot.xacro (robot description, xacro)
@@ -2,5 +2,5 @@
 <robot name="ssl_robot" xmlns:xacro="http://www.ros.org/wiki/xacro">
   <xacro:property name="ground_clearance" value="0.002" />
-  <xacro:property name="base_height" value="0.15" />
+  <xacro:property name="base_height" value="0.138" />
   <xacro:property name="base_radius" value="0.09" />
   <xacro:include filename="$(find ssl_robot_description)/urdf/ssl_robot.gazebo" />
@@ -11,11 +11,7 @@
   <link name="base_plate">
    <inertial>
-      <origin xyz="0 0 ${base_height/2+ground_clearance}" rpy="0 0 0"/>
-<!--
-      <mass value="1.00" />
-      <inertia ixx="0.001233" ixy="0" ixz="0" iyy="0.001233" iyz="0" izz="0.002450" />
--->
-      <mass value="5.00" />
-      <inertia ixx="0.015500" ixy="0" ixz="0" iyy="0.015500" iyz="0" izz="0.012250" />
+      <origin xyz="0 0 0.05" rpy="0 0 0"/>
+      <mass value="34.0" />
+      <inertia ixx="0.15500" ixy="0" ixz="0" iyy="0.15500" iyz="0" izz="0.12250" />
    </inertial>
    <visual>

File: ssl_robot_description/urdf/sub_wheel.xacro (robot description, xacro)
@@ -7,10 +7,6 @@
       <inertial>
         <origin xyz="0 0 0" rpy="0 0 0" />
-<!--
-        <mass value="0.1000" />
-        <inertia ixx="0.0002500521" ixy="0" ixz="0" iyy="0.0002500521" iyz="0" izz="0.0005000000" />
--->
-        <mass value="0.1000" />
-        <inertia ixx="0.0000625521" ixy="0" ixz="0" iyy="0.0000625521" iyz="0" izz="0.0001250000" />
+        <mass value="0.010" />
+        <inertia ixx="0.000000111" ixy="0" ixz="0" iyy="0.000000111" iyz="0" izz="0.000000211" />
       </inertial>
       <collision>

File: ssl_robot_description/urdf/wheel.xacro (robot description, xacro)
@@ -1,5 +1,5 @@
 <?xml version="1.0"?>
 <robot xmlns:xacro="http://www.ros.org/wiki/xacro">
-  <xacro:property name="wheel_radius" value="0.025" />
+  <xacro:property name="wheel_radius" value="0.027" />
   <xacro:property name="wheel_thickness" value="0.015" />
   <xacro:property name="robot_wheel_radius" value="0.075" />
@@ -9,10 +9,6 @@
       <inertial>
         <origin xyz="${wheel_thickness/2} 0 0" rpy="0 1.5707 0" />
-<!--
-        <mass value="0.5000" />
-        <inertia ixx="0.0003218750" ixy="0" ixz="0" iyy="0.0003218750" iyz="0" izz="0.0006250000" />
--->
-        <mass value="0.5000" />
-        <inertia ixx="0.0012593750" ixy="0" ixz="0" iyy="0.0012593750" iyz="0" izz="0.0025000000" />
+        <mass value="0.8000" />
+        <inertia ixx="0.012593750" ixy="0" ixz="0" iyy="0.012593750" iyz="0" izz="0.025000000" />
       </inertial>
       <visual>
@@ -22,4 +18,5 @@
         </geometry>
       </visual>
+<!--
       <collision>
         <origin xyz="${wheel_thickness/2} 0 0" rpy="0 1.5707 0" />
@@ -28,4 +25,5 @@
         </geometry>
       </collision>
+-->
     </link>
     <joint name="base_wheel_${suffix}" type="continuous">
