Commit message: use inertias from real robot (CAD) in gazebo sim

File: ssl_robot_description/urdf/ssl_robot.xacro (robot description, xacro)
@@ -11,11 +11,10 @@
   <link name="base_plate">
    <inertial>
-      <origin xyz="0 0 ${base_height/2+ground_clearance}" rpy="0 0 0"/>
-<!--
-      <mass value="1.00" />
-      <inertia ixx="0.001233" ixy="0" ixz="0" iyy="0.001233" iyz="0" izz="0.002450" />
+      <origin xyz="0 0 0.05" rpy="0 0 0"/>
+<!--		<mass value="5.00" />
+		<inertia ixx="0.121875" ixy="0" ixz="0" iyy="0.121875" iyz="0" izz="0.225000" />
 -->
-      <mass value="5.00" />
-      <inertia ixx="0.015500" ixy="0" ixz="0" iyy="0.015500" iyz="0" izz="0.012250" />
+		<mass value="3.669" />
+		<inertia ixx="0.012646186" ixy="-0.000204481" ixz="-0.000024516" iyy="0.014053275" iyz="-0.000015230" izz="0.015508810" />
    </inertial>
    <visual>

File: ssl_robot_description/urdf/sub_wheel.xacro (robot description, xacro)
@@ -7,10 +7,10 @@
       <inertial>
         <origin xyz="0 0 0" rpy="0 0 0" />
+        <mass value="0.001" />
+        <inertia ixx="0.0000625521" ixy="0" ixz="0" iyy="0.0000625521" iyz="0" izz="0.0001250000" />
 <!--
-        <mass value="0.1000" />
-        <inertia ixx="0.0002500521" ixy="0" ixz="0" iyy="0.0002500521" iyz="0" izz="0.0005000000" />
+        <mass value="0.001" />
+        <inertia ixx="0.000000005" ixy="0" ixz="0" iyy="0.000000005" iyz="0" izz="0.000000008" />
 -->
-        <mass value="0.1000" />
-        <inertia ixx="0.0000625521" ixy="0" ixz="0" iyy="0.0000625521" iyz="0" izz="0.0001250000" />
       </inertial>
       <collision>
@@ -26,5 +26,5 @@
       <axis xyz="0 0 1" />
       <origin xyz="0.007 ${origin_x} ${origin_y}" rpy="${rotation} 0 0" />
-      <dynamics damping="0.0001" friction="0.0" />
+      <dynamics damping="0.001" friction="0.0" />
     </joint>
   </xacro:macro>

File: ssl_robot_description/urdf/wheel.xacro (robot description, xacro)
@@ -11,8 +11,8 @@
 <!--
         <mass value="0.5000" />
-        <inertia ixx="0.0003218750" ixy="0" ixz="0" iyy="0.0003218750" iyz="0" izz="0.0006250000" />
+        <inertia ixx="0.0012593750" ixy="0" ixz="0" iyy="0.0012593750" iyz="0" izz="0.0025000000" />
 -->
-        <mass value="0.5000" />
-        <inertia ixx="0.0012593750" ixy="0" ixz="0" iyy="0.0012593750" iyz="0" izz="0.0025000000" />
+        <mass value="0.1000" />
+        <inertia ixx="0.000018493" ixy="0" ixz="0" iyy="0.000018493" iyz="0" izz="0.000033541" />
       </inertial>
       <visual>
@@ -22,4 +22,5 @@
         </geometry>
       </visual>
+<!--
       <collision>
         <origin xyz="${wheel_thickness/2} 0 0" rpy="0 1.5707 0" />
@@ -28,4 +29,5 @@
         </geometry>
       </collision>
+-->
     </link>
     <joint name="base_wheel_${suffix}" type="continuous">

Commit message: tweaked some gazebo and move_base parameters

File: ssl_robot_description/urdf/ssl_robot.xacro (robot description, xacro)
@@ -11,5 +11,5 @@
   <link name="base_plate">
    <inertial>
-      <origin xyz="0 0 0.05" rpy="0 0 0"/>
+      <origin xyz="0 0 0.03" rpy="0 0 0"/>
       <mass value="34.0" />
       <inertia ixx="0.15500" ixy="0" ixz="0" iyy="0.15500" iyz="0" izz="0.12250" />

File: ssl_robot_description/urdf/sub_wheel.xacro (robot description, xacro)
@@ -22,5 +22,5 @@
       <axis xyz="0 0 1" />
       <origin xyz="0.007 ${origin_x} ${origin_y}" rpy="${rotation} 0 0" />
-      <dynamics damping="0.0001" friction="0.0" />
+      <dynamics damping="0.0001" friction="0.1" />
     </joint>
   </xacro:macro>

File: ssl_robot_description/urdf/wheel.xacro (robot description, xacro)
@@ -32,5 +32,5 @@
       <axis xyz="1 0 0" />
       <origin xyz="${robot_wheel_radius*origin_x} ${robot_wheel_radius*origin_y} ${wheel_radius-ground_clearance}" rpy="0 0 ${rotation}" />
-      <dynamics damping="0.05" friction="0.0" />
+      <dynamics damping="0.05" friction="0.1" />
       <!-- (3m/s / 2*pi*r) * 2 * pi -> 3m/s / r-->
       <limit lower="0" upper="0"
